File: espkit-01.kicad_pcb (KiCad board)
At the start: 2 copper layers, 41.8 x 25 mm, 29 parts, among them IC1 WS2812B, P1 ESP-01, P2 BREAKOUT, P2 CONN_7, P3 SERIAL, P4 PWR, P5 NEOPIXEL, P6 BRIDGE, SW1 RESET, SW2 PRGM

Commit message: Updated text.
Other:
- board text added: "ESPkit-01 V1.0 https://github.com/mage0r/ESPkit-01 John Spencer & Andy Gelme, 2015 Made at hackmelbourne.org"
- board text removed: "LearnESP-01 V1.0 https://github.com/mage0r/LearnESP-01 John Spencer & Andy Gelme, 2015 Made at hackmelbourne.org"
Changed lines of the file:
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@@
     (effects (font (size 0.5 0.5) (thickness 0.1)))
   )
-  (gr_text "LearnESP-01 V1.0\nhttps://github.com/mage0r/LearnESP-01\nJohn Spencer & Andy Gelme, 2015\nMade at hackmelbourne.org" (at 44 34.3) (layer F.SilkS)
+  (gr_text "ESPkit-01 V1.0\nhttps://github.com/mage0r/ESPkit-01\nJohn Spencer & Andy Gelme, 2015\nMade at hackmelbourne.org" (at 44 34.3) (layer F.SilkS)
     (effects (font (size 0.4 0.4) (thickness 0.1)))
   )
@@
   (gr_arc (start 12.4 12.4) (end 12.1 12.4) (angle 90) (layer Edge.Cuts) (width 0.1))
   (gr_arc (start 12.4 36.8) (end 12.4 37.1) (angle 90) (layer Edge.Cuts) (width 0.1))
-  (gr_text "LearnESP-01 V1.0\nhttps://github.com/mage0r/LearnESP-01\nJohn Spencer & Andy Gelme, 2015\nMade at hackmelbourne.org" (at 22.2 34.3) (layer F.SilkS)
+  (gr_text "ESPkit-01 V1.0\nhttps://github.com/mage0r/ESPkit-01\nJohn Spencer & Andy Gelme, 2015\nMade at hackmelbourne.org" (at 22.2 34.3) (layer F.SilkS)
     (effects (font (size 0.4 0.4) (thickness 0.1)))
   )

Commit message: Added single layer version
or, at least, as single as possible.  There are 4 connections on the
back, but they are between pins.
Parts:
- removed the C2 at (52.9, 18.0)
- removed the C3 at (52.9, 14.6)
- removed the D1 at (34.9, 14.8)
- removed the IC1 at (44.1, 19.9)
- removed the P1 at (44.0, 28.3)
- removed the P2 at (36.1, 27.5)
- removed the P2 at (33.0, 23.8)
- removed the P3 at (44.0, 14.4)
- removed the P4 at (36.1, 32.9)
- removed the P5 at (51.8, 30.4)
- removed the P6 at (44.2, 23.4)
- removed the R1 at (52.9, 21.4)
- removed the R3 at (35.0, 18.4)
- removed the SW1 at (50.1, 19.9)
- removed the SW2 at (38.0, 19.9)
Routing:
- net GND: track 156.4 -> 73.3 mm
- net +3.3V: track 140.0 -> 105.7 mm, vias 2 -> 0
- net GPIO2: track 56.0 -> 30.5 mm
- net RX: track 38.9 -> 21.9 mm
- net GPIO0: track 31.2 -> 14.8 mm
- net TX: track 27.4 -> 13.7 mm
- net N-0000011: track 29.6 -> 20.1 mm, vias 2 -> 0
- net N-000005: track 3.28 -> 1.64 mm
Other:
- board size 41.8 x 25 mm -> 20 x 25 mm

Commit message: Shuffled Layout for 1.1
Parts:
- C3: value 10uf -> 1uf
- moved C3 13.3 mm to (18.7, 19.3), turned to 0 degrees
- moved C2 12.8 mm to (18.7, 21.3), turned to 0 degrees
- moved R1 7.20 mm to (31.0, 14.2)
- moved R3 5.61 mm to (18.7, 17.3), turned to 0 degrees
- moved SW2 2.16 mm to (14.1, 20.4)
- moved IC1 1.94 mm to (24.2, 19.5)
- moved SW1 1.87 mm to (30.1, 20.4), turned to 90 degrees
- moved P6 1.77 mm to (24.1, 22.9)
- moved P2 1.60 mm to (14.4, 29.1), turned to 90 degrees
- moved P4 1.30 mm to (14.4, 34.2)
- moved P5 1.30 mm to (30.0, 31.7)
- moved D1 0.98 mm to (13.5, 13.9)
- moved P1 0.91 mm to (22.3, 27.4)
Connections:
- IC1 pad 4: GPIO2 -> N-000004
- P1 pad 1: RX -> TX
- P1 pad 8: TX -> RX
- P4 pad 1: +3.3V -> GND
- P4 pad 2: GND -> +3.3V
- P6 pad 1: GPIO2 -> N-000004
Routing:
- net +3.3V: track 105.7 -> 64.1 mm
- net RX: track 21.9 -> 13.2 mm
- net GPIO2: track 30.5 -> 24.5 mm
- net N-0000012: track 20.1 -> 24.9 mm
- net N-000006: track 1.64 -> 5.31 mm
- net N-000004: track 0.00 -> 3.42 mm
- net GND: track 73.3 -> 70.1 mm
- net TX: track 13.7 -> 16.8 mm
Other:
- board text added: "Bridge for PRGM"
- board text added: "ESPkit-01 V1.1 https://github.com/mage0r/ESPkit-01 John Spencer & Andy Gelme, 2015 Made at hackmelbourne.org"
- board text removed: "ESPkit-01 V1.0 https://github.com/mage0r/ESPkit-01 John Spencer & Andy Gelme, 2015 Made at hackmelbourne.org"
